File: 01_MainCircuitry.kicad_sch (KiCad schematic)
At the start: 20 parts, among them Q1 Q_NMOS, Q2 Q_NMOS, Q3 Q_NMOS, Q4 Q_NMOS, Q5 Q_NMOS, Q6 Q_NMOS

Commit message: small change to 01 main circuit
Connections:
- net +48V: now also Q1.D, Q3.D, Q5.D
Changed lines of the file:
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@@
-	)
-	(junction
-		(at 130.81 81.28)
-		(diameter 0)
-		(color 0 0 0 0)
 	)
 	(junction
@@
 	(wire
 		(pts
-			(xy 31.75 63.5) (xy 31.75 62.23)
-		)
-		(stroke
-			(width 0)
-			(type default)
-		)
-	)
-	(wire
-		(pts
 			(xy 162.56 81.28) (xy 162.56 86.36)
 		)
@@
 	(wire
 		(pts
+			(xy 31.75 49.53) (xy 31.75 43.18)
+		)
+		(stroke
+			(width 0)
+			(type default)
+		)
+	)
+	(wire
+		(pts
 			(xy 97.79 49.53) (xy 97.79 66.04)
 		)
@@
 	(wire
 		(pts
-			(xy 129.54 81.28) (xy 130.81 81.28)
+			(xy 130.81 81.28) (xy 135.89 81.28)
 		)
 		(stroke
@@
 	(wire
 		(pts
-			(xy 33.02 63.5) (xy 31.75 63.5)
-		)
-		(stroke
-			(width 0)
-			(type default)
-		)
-	)
-	(wire
-		(pts
 			(xy 162.56 81.28) (xy 201.93 81.28)
 		)
@@
 	(wire
 		(pts
-			(xy 31.75 59.69) (xy 31.75 49.53)
-		)
-		(stroke
-			(width 0)
-			(type default)
-		)
-	)
-	(wire
-		(pts
 			(xy 40.64 49.53) (xy 68.58 49.53)
 		)
@@
 		(pts
 			(xy 114.3 96.52) (xy 114.3 101.6)
-		)
-		(stroke
-			(width 0)
-			(type default)
-		)
-	)
-	(wire
-		(pts
-			(xy 130.81 81.28) (xy 135.89 81.28)
 		)
 		(stroke
@@
 	(symbol
 		(lib_id "power:+48V")
-		(at 31.75 62.23 0)
+		(at 31.75 43.18 0)
 		(unit 1)
 		(exclude_from_sim no)
@@
 		(fields_autoplaced yes)
 		(property "Reference" "#PWR01"
-			(at 31.75 66.04 0)
+			(at 31.75 46.99 0)
 			(effects
 				(font
@@
 		)
 		(property "Value" "+48V"
-			(at 31.75 57.15 0)
+			(at 31.75 38.1 0)
 			(effects
 				(font
@@
 		)
 		(property "Footprint" ""
-			(at 31.75 62.23 0)
+			(at 31.75 43.18 0)
 			(effects
 				(font
@@
 		)
 		(property "Datasheet" ""
-			(at 31.75 62.23 0)
+			(at 31.75 43.18 0)
 			(effects
 				(font
@@
 		)
 		(property "Description" "Power symbol creates a global label with name \"+48V\""
-			(at 31.75 62.23 0)
+			(at 31.75 43.18 0)
 			(effects
 				(font

Commit message: added some kind of PCB design, a rough draft
Parts:
- C1, Q1, Q6, R1, SR1, SR2, SR3: now left out of the parts list
- LpA1: renamed from LpA; now left out of the parts list
- LpB1: renamed from LpB; now left out of the parts list
- LpC1: renamed from LpC; now left out of the parts list
- LsA1: renamed from LsA; now left out of the parts list
- LsB1: renamed from LsB; now left out of the parts list
- LsC1: renamed from LsC; now left out of the parts list
- LsOutA1: renamed from LsOutA; now left out of the parts list
- LsOutB1: renamed from LsOutB; now left out of the parts list
- LsOutC1: renamed from LsOutC; now left out of the parts list
- Q2: renamed from Q3; now left out of the parts list
- Q3: renamed from Q5; now left out of the parts list
- Q4: renamed from Q2; now left out of the parts list
- Q5: renamed from Q4; now left out of the parts list
Changed lines of the file:
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@@
 		(at 66.04 113.03 0)
 		(unit 1)
-		(exclude_from_sim no)
-		(in_bom yes)
-		(on_board yes)
-		(dnp no)
-		(fields_autoplaced yes)
-		(property "Reference" "Q4"
+		(exclude_from_sim yes)
+		(in_bom no)
+		(on_board no)
+		(dnp no)
+		(fields_autoplaced yes)
+		(property "Reference" "Q5"
 			(at 72.39 111.7599 0)
 			(effects
@@
 			(project "BachelorCurrentTripler"
 				(path "/eaeaab39-7712-4bb8-8f1a-3ddca096a313/e39cac19-8597-4e40-9e6f-88d9f4803cf9"
-					(reference "Q4")
+					(reference "Q5")
 					(unit 1)
 				)
@@
 		(at 31.75 43.18 0)
 		(unit 1)
-		(exclude_from_sim no)
-		(in_bom yes)
-		(on_board yes)
-		(dnp no)
-		(fields_autoplaced yes)
-		(property "Reference" "#PWR01"
+		(exclude_from_sim yes)
+		(in_bom no)
+		(on_board no)
+		(dnp no)
+		(fields_autoplaced yes)
+		(property "Reference" "#PWR03"
 			(at 31.75 46.99 0)
 			(effects
@@
 			(project ""
 				(path "/eaeaab39-7712-4bb8-8f1a-3ddca096a313/e39cac19-8597-4e40-9e6f-88d9f4803cf9"
-					(reference "#PWR01")
+					(reference "#PWR03")
 					(unit 1)
 				)
@@
 		(at 127 91.44 90)
 		(unit 1)
-		(exclude_from_sim no)
-		(in_bom yes)
-		(on_board yes)
-		(dnp no)
-		(fields_autoplaced yes)
-		(property "Reference" "LpB"
+		(exclude_from_sim yes)
+		(in_bom no)
+		(on_board no)
+		(dnp no)
+		(fields_autoplaced yes)
+		(property "Reference" "LpB1"
 			(at 127 86.36 90)
 			(effects
@@
 			(project "BachelorCurrentTripler"
 				(path "/eaeaab39-7712-4bb8-8f1a-3ddca096a313/e39cac19-8597-4e40-9e6f-88d9f4803cf9"
-					(reference "LpB")
+					(reference "LpB1")
 					(unit 1)
 				)
@@
 		(at 35.56 132.08 0)
 		(unit 1)
-		(exclude_from_sim no)
-		(in_bom yes)
-		(on_board yes)
-		(dnp no)
-		(fields_autoplaced yes)
-		(property "Reference" "#PWR02"
+		(exclude_from_sim yes)
+		(in_bom no)
+		(on_board no)
+		(dnp no)
+		(fields_autoplaced yes)
+		(property "Reference" "#PWR04"
 			(at 35.56 138.43 0)
 			(effects
@@
 			(project ""
 				(path "/eaeaab39-7712-4bb8-8f1a-3ddca096a313/e39cac19-8597-4e40-9e6f-88d9f4803cf9"
-					(reference "#PWR02")
+					(reference "#PWR04")
 					(unit 1)
 				)
@@
 		(at 127 101.6 90)
 		(unit 1)
-		(exclude_from_sim no)
-		(in_bom yes)
-		(on_board yes)
-		(dnp no)
-		(fields_autoplaced yes)
-		(property "Reference" "LpC"
+		(exclude_from_sim yes)
+		(in_bom no)
+		(on_board no)
+		(dnp no)
+		(fields_autoplaced yes)
+		(property "Reference" "LpC1"
 			(at 127 96.52 90)
 			(effects
@@
 			(project "BachelorCurrentTripler"
 				(path "/eaeaab39-7712-4bb8-8f1a-3ddca096a313/e39cac19-8597-4e40-9e6f-88d9f4803cf9"
-					(reference "LpC")
+					(reference "LpC1")
 					(unit 1)
 				)
@@
 		(at 95.25 71.12 0)
 		(unit 1)
-		(exclude_from_sim no)
-		(in_bom yes)
-		(on_board yes)
-		(dnp no)
-		(fields_autoplaced yes)
-		(property "Reference" "Q5"
+		(exclude_from_sim yes)
+		(in_bom no)
+		(on_board no)
+		(dnp no)
+		(fields_autoplaced yes)
+		(property "Reference" "Q3"
 			(at 101.6 69.8499 0)
 			(effects
@@
 			(project "BachelorCurrentTripler"
 				(path "/eaeaab39-7712-4bb8-8f1a-3ddca096a313/e39cac19-8597-4e40-9e6f-88d9f4803cf9"
-					(reference "Q5")
+					(reference "Q3")
 					(unit 1)
 				)
@@
 		(at 180.34 52.07 0)
 		(unit 1)
-		(exclude_from_sim no)
-		(in_bom yes)
-		(on_board yes)
-		(dnp no)
-		(fields_autoplaced yes)
-		(property "Reference" "LsOutA"
+		(exclude_from_sim yes)
+		(in_bom no)
+		(on_board no)
+		(dnp no)
+		(fields_autoplaced yes)
+		(property "Reference" "LsOutA1"
 			(at 181.61 50.7999 0)
 			(effects
@@
 			(project ""
 				(path "/eaeaab39-7712-4bb8-8f1a-3ddca096a313/e39cac19-8597-4e40-9e6f-88d9f4803cf9"
-					(reference "LsOutA")
+					(reference "LsOutA1")
 					(unit 1)
 				)
@@
 		(at 162.56 90.17 0)
 		(unit 1)
-		(exclude_from_sim no)
-		(in_bom yes)
-		(on_board yes)
-		(dnp no)
-		(fields_autoplaced yes)
-		(property "Reference" "LsB"
+		(exclude_from_sim yes)
+		(in_bom no)
+		(on_board no)
+		(dnp no)
+		(fields_autoplaced yes)
+		(property "Reference" "LsB1"
 			(at 163.83 88.8999 0)
 			(effects
@@
 			(project "BachelorCurrentTripler"
 				(path "/eaeaab39-7712-4bb8-8f1a-3ddca096a313/e39cac19-8597-4e40-9e6f-88d9f4803cf9"
-					(reference "LsB")
+					(reference "LsB1")
 					(unit 1)
 				)
@@
 		(at 219.71 118.11 0)
 		(unit 1)
-		(exclude_from_sim no)
-		(in_bom yes)
-		(on_board yes)
+		(exclude_from_sim yes)
+		(in_bom no)
+		(on_board no)
 		(dnp no)
 		(fields_autoplaced yes)
@@
 		(at 95.25 113.03 0)
 		(unit 1)
-		(exclude_from_sim no)
-		(in_bom yes)
-		(on_board yes)
+		(exclude_from_sim yes)
+		(in_bom no)
+		(on_board no)
 		(dnp no)
 		(fields_autoplaced yes)
@@
 		(at 38.1 113.03 0)
 		(unit 1)
-		(exclude_from_sim no)
-		(in_bom yes)
-		(on_board yes)
-		(dnp no)
-		(fields_autoplaced yes)
-		(property "Reference" "Q2"
+		(exclude_from_sim yes)
+		(in_bom no)
+		(on_board no)
+		(dnp no)
+		(fields_autoplaced yes)
+		(property "Reference" "Q4"
 			(at 44.45 111.7599 0)
 			(effects
@@
 			(project ""
 				(path "/eaeaab39-7712-4bb8-8f1a-3ddca096a313/e39cac19-8597-4e40-9e6f-88d9f4803cf9"
-					(reference "Q2")
+					(reference "Q4")
 					(unit 1)
 				)
@@
 		(at 199.39 118.11 0)
 		(unit 1)
-		(exclude_from_sim no)
-		(in_bom yes)
-		(on_board yes)
+		(exclude_from_sim yes)
+		(in_bom no)
+		(on_board no)
 		(dnp no)
 		(property "Reference" "SR2"
@@
 		(at 177.8 118.11 0)
 		(unit 1)
-		(exclude_from_sim no)
-		(in_bom yes)
-		(on_board yes)
+		(exclude_from_sim yes)
+		(in_bom no)
+		(on_board no)
 		(dnp no)
 		(fields_autoplaced yes)
@@
 		(at 265.43 85.09 0)
 		(unit 1)
-		(exclude_from_sim no)
-		(in_bom yes)
-		(on_board yes)
+		(exclude_from_sim yes)
+		(in_bom no)
+		(on_board no)
 		(dnp no)
 		(fields_autoplaced yes)
@@
 		(at 38.1 71.12 0)
 		(unit 1)
-		(exclude_from_sim no)
-		(in_bom yes)
-		(on_board yes)
+		(exclude_from_sim yes)
+		(in_bom no)
+		(on_board no)
 		(dnp no)
 		(fields_autoplaced yes)
@@
 		(at 148.59 90.17 180)
 		(unit 1)
-		(exclude_from_sim no)
-		(in_bom yes)
-		(on_board yes)
-		(dnp no)
-		(fields_autoplaced yes)
-		(property "Reference" "LsC"
+		(exclude_from_sim yes)
+		(in_bom no)
+		(on_board no)
+		(dnp no)
+		(fields_autoplaced yes)
+		(property "Reference" "LsC1"
 			(at 149.86 88.8999 0)
 			(effects
@@
 			(project "BachelorCurrentTripler"
 				(path "/eaeaab39-7712-4bb8-8f1a-3ddca096a313/e39cac19-8597-4e40-9e6f-88d9f4803cf9"
-					(reference "LsC")
+					(reference "LsC1")
 					(unit 1)
 				)
@@
 		(at 156.21 81.28 90)
 		(unit 1)
-		(exclude_from_sim no)
-		(in_bom yes)
-		(on_board yes)
-		(dnp no)
-		(fields_autoplaced yes)
-		(property "Reference" "LsA"
+		(exclude_from_sim yes)
+		(in_bom no)
+		(on_board no)
+		(dnp no)
+		(fields_autoplaced yes)
+		(property "Reference" "LsA1"
 			(at 156.21 76.2 90)
 			(effects
@@
 			(project "BachelorCurrentTripler"
 				(path "/eaeaab39-7712-4bb8-8f1a-3ddca096a313/e39cac19-8597-4e40-9e6f-88d9f4803cf9"
-					(reference "LsA")
+					(reference "LsA1")
 					(unit 1)
 				)
@@
 		(at 201.93 52.07 0)
 		(unit 1)
-		(exclude_from_sim no)
-		(in_bom yes)
-		(on_board yes)
-		(dnp no)
-		(fields_autoplaced yes)
-		(property "Reference" "LsOutB"
+		(exclude_from_sim yes)
+		(in_bom no)
+		(on_board no)
+		(dnp no)
+		(fields_autoplaced yes)
+		(property "Reference" "LsOutB1"
 			(at 203.2 50.7999 0)
 			(effects
@@
 			(project ""
 				(path "/eaeaab39-7712-4bb8-8f1a-3ddca096a313/e39cac19-8597-4e40-9e6f-88d9f4803cf9"
-					(reference "LsOutB")
+					(reference "LsOutB1")
 					(unit 1)
 				)
@@
 		(at 66.04 71.12 0)
 		(unit 1)
-		(exclude_from_sim no)
-		(in_bom yes)
-		(on_board yes)
-		(dnp no)
-		(fields_autoplaced yes)
-		(property "Reference" "Q3"
+		(exclude_from_sim yes)
+		(in_bom no)
+		(on_board no)
+		(dnp no)
+		(fields_autoplaced yes)
+		(property "Reference" "Q2"
 			(at 72.39 69.8499 0)
 			(effects
@@
 			(project ""
 				(path "/eaeaab39-7712-4bb8-8f1a-3ddca096a313/e39cac19-8597-4e40-9e6f-88d9f4803cf9"
-					(reference "Q3")
+					(reference "Q2")
 					(unit 1)
 				)
@@
 		(at 240.03 85.09 0)
 		(unit 1)
-		(exclude_from_sim no)
-		(in_bom yes)
-		(on_board yes)
+		(exclude_from_sim yes)
+		(in_bom no)
+		(on_board no)
 		(dnp no)
 		(fields_autoplaced yes)
@@
 		(at 222.25 52.07 0)
 		(unit 1)
-		(exclude_from_sim no)
-		(in_bom yes)
-		(on_board yes)
-		(dnp no)
-		(fields_autoplaced yes)
-		(property "Reference" "LsOutC"
+		(exclude_from_sim yes)
+		(in_bom no)
+		(on_board no)
+		(dnp no)
+		(fields_autoplaced yes)
+		(property "Reference" "LsOutC1"
 			(at 223.52 50.7999 0)
 			(effects
@@
 			(project "BachelorCurrentTripler"
 				(path "/eaeaab39-7712-4bb8-8f1a-3ddca096a313/e39cac19-8597-4e40-9e6f-88d9f4803cf9"
-					(reference "LsOutC")
+					(reference "LsOutC1")
 					(unit 1)
 				)
@@
 		(at 127 81.28 90)
 		(unit 1)
-		(exclude_from_sim no)
-		(in_bom yes)
-		(on_board yes)
-		(dnp no)
-		(fields_autoplaced yes)
-		(property "Reference" "LpA"
+		(exclude_from_sim yes)
+		(in_bom no)
+		(on_board no)
+		(dnp no)
+		(fields_autoplaced yes)
+		(property "Reference" "LpA1"
 			(at 127 76.2 90)
 			(effects
@@
 			(project ""
 				(path "/eaeaab39-7712-4bb8-8f1a-3ddca096a313/e39cac19-8597-4e40-9e6f-88d9f4803cf9"
-					(reference "LpA")
-					(unit 1)
-				)
+					(reference "LpA1")
+					(unit 1)
+				)
