File: BachelorCurrentTripler.kicad_sch (KiCad schematic)
At the start: 5 parts, among them J1 Conn_01x07_Pin, J2 Conn_01x01_Pin, J3 Conn_01x01_Pin, J4 Conn_01x04_Socket, J5 Conn_01x01_Pin

Commit message: Secondary side finished
Parts:
- added C36, C37: C, Capacitor_THT:CP_Radial_D8.0mm_P5.00mm, symbol Device:C
Connections:
- net +12V: now also C36.1
- net +48V: now also C37.1
- net GND: now also C36.2, C37.2

Commit message: Rettelser efter møde med Andreas
Parts:
- added H1, H2, H3, H4: MountingHole_Pad, MountingHole:MountingHole_4.3mm_M4_Pad_Via, symbol Mechanical:MountingHole_Pad
Connections:
- net GND: now also H1.1, H2.1, H3.1, H4.1
